Commit message: odom+joint modified

File: charlie/urdf/test.urdf.xacro (robot description, xacro)
@@ -9,5 +9,5 @@
     <parent link="base_footprint"/>
     <child link="base_link" />
-    <origin xyz="0 0 0.010" rpy="0 0 0"/>
+    <origin xyz="0 0 0.010" rpy="0 0 3.14"/>
   </joint>
   <link name="base_link">

Commit message: add imu

File: charlie/urdf/test.urdf.xacro (robot description, xacro)
@@ -9,5 +9,5 @@
     <parent link="base_footprint"/>
     <child link="base_link" />
-    <origin xyz="0 0 0.010" rpy="0 0 3.14"/>
+    <origin xyz="0 0 0.010" rpy="0 0 0"/>
   </joint>
   <link name="base_link">
@@ -126,8 +126,9 @@
     </inertial>
   </link>
+  	<!--
   <joint name="imu_joint" type="fixed">
     <parent link="base_link"/>
     <child link="imu_link"/>
-    <origin xyz="0.0 0 0.068" rpy="0 0 0"/>
+    <origin xyz="0 0 0" rpy="0 0 0"/>
   </joint>
   <link name="imu_link"/>
@@ -135,5 +136,5 @@
     <parent link="base_link"/>
     <child link="base_scan"/>
-    <origin xyz="-0.064 0 0.1" rpy="0 0 0"/>
+    <origin xyz="0 0 0" rpy="0 0 0"/>
   </joint>
   <link name="base_scan">
@@ -151,4 +152,5 @@
     </collision>
   </link>
+  	-->
   <!-- Camera and other components can be added here -->
 </robot>

Commit message: gmapping

File: charlie/urdf/test.urdf.xacro (robot description, xacro)
@@ -89,5 +89,5 @@
     <parent link="base_link"/>
     <child link="caster_back_right_link"/>
-    <origin xyz="-0.177 -0.064 -0.004" rpy="-1.57 0 0"/>
+    <origin xyz="-0.38 -0.15 -0.004" rpy="-1.57 0 0"/>
   </joint>
   <link name="caster_back_right_link">
@@ -109,5 +109,5 @@
     <parent link="base_link"/>
     <child link="caster_back_left_link"/>
-    <origin xyz="-0.177 0.064 -0.004" rpy="-1.57 0 0"/>
+    <origin xyz="-0.38 0.15 -0.004" rpy="-1.57 0 0"/>
   </joint>
   <link name="caster_back_left_link">
@@ -133,8 +133,9 @@
   </joint>
   <link name="imu_link"/>
+  -->
   <joint name="scan_joint" type="fixed">
     <parent link="base_link"/>
     <child link="base_scan"/>
-    <origin xyz="0 0 0" rpy="0 0 0"/>
+    <origin xyz="0 0 0.25" rpy="0 0 0"/>
   </joint>
   <link name="base_scan">
@@ -152,5 +153,4 @@
     </collision>
   </link>
-  	-->
   <!-- Camera and other components can be added here -->
 </robot>
